Commit message: changes done

File: urdf/edrone_model.urdf (robot description, URDF)
Before this commit: robot edrone_model, 9 links, 8 joints
Links:
- removed link caster_b_link
- removed link caster_back_link
- removed link caster_front_link
- removed link caster_link
- removed link left_wheel
- removed link middle_link
- removed link right_wheel
- removed link top_link
- added link holder_link, mass .2; collision mesh filename=package://edrone_gazebo/urdf/stl/holder.stl scale=0.05 0.05 0.05; visual mesh filename=package://edrone_gazebo/urdf/stl/holder.stl scale=0.1 0.1 0.1
- link frame_link: geometry collision mesh filename=package://edrone_gazebo/urdf/stl/frame.stl scale=0.1 0.1 0.1; visual mesh filename=package://edrone_gazebo/urdf/stl/frame.stl scale=0.1 0.1 0.1
Joints:
- removed joint caster_back_joint
- removed joint caster_back_joint_base
- removed joint caster_front_joint
- removed joint caster_front_joint_base
- removed joint left_wheel_joint
- removed joint right_wheel_joint
- removed joint top_joint
- joint middle_joint: child middle_link -> holder_link; origin xyz=0 0.0 .07 rpy=0 0 0 -> xyz=0 0 0 rpy=0 0 0

Commit message: changes in urdf file

File: urdf/edrone_model.urdf (robot description, URDF)
Before this commit: robot edrone_model, 2 links, 1 joints
Links:
- removed link frame_link
- removed link holder_link
- added link base_link
- added link base_link_inertia, mass 0.0085; collision box size=0.14 0.14 0.015; visual mesh filename=package://edrone_gazebo/urdf/stl/frame.stl scale=0.001 0.001 0.001
- added link rotor_0, mass 0.0037; collision cylinder length=0.005 radius=0.0035; visual mesh filename=package://edrone_gazebo/urdf/stl/prop_CCW_45.stl scale=0.001 0.001 0.001
- added link rotor_1, mass 0.0037; collision cylinder length=0.005 radius=0.0035; visual mesh filename=package://edrone_gazebo/urdf/stl/prop_CW_45.stl scale=0.001 0.001 0.001
- added link rotor_2, mass 0.0037; collision cylinder length=0.005 radius=0.0035; visual mesh filename=package://edrone_gazebo/urdf/stl/prop_CCW_45.stl scale=0.001 0.001 0.001
- added link rotor_3, mass 0.0037; collision cylinder length=0.005 radius=0.0035; visual mesh filename=package://edrone_gazebo/urdf/stl/prop_CW_45.stl scale=0.001 0.001 0.001
Joints:
- removed joint middle_joint
- added joint base_joint: type fixed, parent base_link, child base_link_inertia, origin xyz=0 0 0 rpy=0 0 0
- added joint rotor_0_joint: type continuous, parent base_link, child rotor_0, origin xyz=0.0675 0 0.01 rpy=0 0 0, axis 0 0 1
- added joint rotor_1_joint: type continuous, parent base_link, child rotor_1, origin xyz=0 -0.0675 0.01 rpy=0 0 0, axis 0 0 1
- added joint rotor_2_joint: type continuous, parent base_link, child rotor_2, origin xyz=-0.0675 0 0.01 rpy=0 0 0, axis 0 0 1
- added joint rotor_3_joint: type continuous, parent base_link, child rotor_3, origin xyz=0 0.0675 0.01 rpy=0 0 0, axis 0 0 1

Commit message: little changes

File: urdf/edrone_model.urdf (robot description, URDF)
Before this commit: robot edrone_model, 9 links, 8 joints
Links:
- removed link caster_b_link
- removed link caster_back_link
- removed link caster_front_link
- removed link caster_link
- removed link left_wheel
- removed link middle_link
- removed link right_wheel
- removed link top_link
- added link holder_link, mass .2; collision mesh filename=package://edrone_gazebo/urdf/stl/holder.stl scale=0.01 0.01 0.01; visual mesh filename=package://edrone_gazebo/urdf/stl/holder.stl scale=0.01 0.01 0.01
- link frame_link: geometry collision mesh filename=package://edrone_gazebo/urdf/stl/frame.stl scale=0.01 0.01 0.01; visual mesh filename=package://edrone_gazebo/urdf/stl/frame.stl scale=0.01 0.01 0.01
Joints:
- removed joint caster_back_joint
- removed joint caster_back_joint_base
- removed joint caster_front_joint
- removed joint caster_front_joint_base
- removed joint left_wheel_joint
- removed joint right_wheel_joint
- removed joint top_joint
- joint middle_joint: child middle_link -> holder_link; origin xyz=0 0.0 .07 rpy=0 0 0 -> xyz=0 0 0 rpy=0 0 0

Commit message: inertia and mesh file rectified

File: urdf/edrone_model.urdf (robot description, URDF)
Before this commit: robot edrone_gazebo, 6 links, 5 joints
Links:
- link base_link_inertia: geometry collision box size=0.14 0.14 0.015; visual mesh filename=package://edrone_gazebo/urdf/meshes/frame.dae scale=0.001 0.001 0.001
- link rotor_0: geometry collision cylinder length=0.005 radius=0.0035; visual mesh filename=package://edrone_gazebo/urdf/meshes/prop_CCW_45.dae scale=0.001 0.001 0.001
- link rotor_1: geometry collision cylinder length=0.005 radius=0.0035; visual mesh filename=package://edrone_gazebo/urdf/meshes/prop_CW_45.dae scale=0.001 0.001 0.001
- link rotor_2: geometry collision cylinder length=0.005 radius=0.0035; visual mesh filename=package://edrone_gazebo/urdf/meshes/prop_CCW_45.dae scale=0.001 0.001 0.001
- link rotor_3: geometry collision cylinder length=0.005 radius=0.0035; visual mesh filename=package://edrone_gazebo/urdf/meshes/prop_CW_45.dae scale=0.001 0.001 0.001

File: urdf/edrone_model.urdf.xacro (robot description, xacro)
@@ -4,8 +4,8 @@
   <xacro:property name="namespace" value="edrone_gazebo" />
   <xacro:property name="rotor_velocity_slowdown_sim" value="10" />
-  <xacro:property name="mesh_file" value="frame.stl" />
+  <xacro:property name="mesh_file" value="frame.dae" />
   <xacro:property name="mesh_scale" value="0.001 0.001 0.001"/>
   <xacro:property name="mesh" value="prop"/>  <!-- "propeller" -->
-  <xacro:property name="mesh_scale_prop" value="0.12 0.12 0.12"/>
+  <xacro:property name="mesh_scale_prop" value="0.001 0.001 0.001"/>
   <xacro:property name="mass" value="0.0085" /> <!-- [kg] -->
   <xacro:property name="body_width" value="0.14" /> <!-- [m] -->
@@ -109,5 +109,5 @@
     mesh="prop"
     mesh_scale="${mesh_scale_prop}"
-    color="Grey">
+    color="black">
     <origin xyz="-${arm_length} 0 ${rotor_offset_top}" rpy="0 0 0" />
     <xacro:insert_block name="rotor_inertia" />

File: urdf/multirotor_base.xacro (robot description, xacro)
@@ -82,5 +82,5 @@
           <!-- <cylinder length="0.005" radius="${radius_rotor}"/> --> <!-- [m] -->
           <!-- <mesh filename="package://rotors_description/meshes/propeller_${direction}.dae" -->
-          <mesh filename="package://urdf/meshes/${mesh}_${direction}.stl"
+          <mesh filename="package://urdf/meshes/${mesh}_${direction}.dae"
             scale="${mesh_scale}" />
           <!-- <box size="${2*radius_rotor} 0.01 0.005"/> -->

Commit message: Rotor inertial's postioning and orientation corrected, collision need correction

File: urdf/edrone_model.urdf (robot description, URDF)
Before this commit: robot edrone_gazebo, 6 links, 5 joints
Joints:
- joint rotor_0_joint: origin xyz=0.0675 -0.0675 0.01 rpy=0 0 0 -> xyz=0.046 -0.046 0.0125 rpy=0 0 0
- joint rotor_1_joint: origin xyz=-0.0675 -0.0675 0.01 rpy=0 0 0 -> xyz=-0.046 -0.046 0.0125 rpy=0 0 0
- joint rotor_2_joint: origin xyz=-0.0675 0.0675 0.01 rpy=0 0 0 -> xyz=-0.046 0.046 0.0125 rpy=0 0 0
- joint rotor_3_joint: origin xyz=0.0675 0.0675 0.01 rpy=0 0 0 -> xyz=0.046 0.046 0.0125 rpy=0 0 0

Commit message: marker gazebo model added

File: urdf/edrone_model.urdf (robot description, URDF)
Before this commit: robot edrone_gazebo, 6 links, 5 joints
Joints:
- joint rotor_0_joint: parent base_link -> base_link_inertia
- joint rotor_1_joint: parent base_link -> base_link_inertia
- joint rotor_2_joint: parent base_link -> base_link_inertia
- joint rotor_3_joint: parent base_link -> base_link_inertia
